File: KiCad/robot.sch (KiCad schematic (older format))
At the start: 62 parts, among them Q1 NPN, Q2 NPN, Q3 Q_PMOS, Q4 Q_NPN, Q5 Q_NMOS, Q6 Q_NPN, SW1 SWITCH_INV, SW2 switch_push

Commit message: popravljeni pini
Parts:
- removed D2: LED_R, symbol LED_Small
- removed D3: LED_Z, symbol LED_Small
- removed Q4, Q6: Q_NPN, symbol Q_NPN_BCE
- removed R19, R20: 10k, symbol R
- removed R25, R28: 300, symbol R_Small
- renumbered Q5 to Q4, R21 to R19, R22 to R20, R23 to R21, R24 to R22, R26 to R23, R27 to R24
Connections:
- net BTRX: now also ArduinoMicro1.25 (A4); no longer ArduinoMicro1.2 (SS)
- net BTTX: now also ArduinoMicro1.16 (D11); no longer ArduinoMicro1.33 (MISO)
- net C1: now also ArduinoMicro1.26 (A5); no longer ArduinoMicro1.16 (D11)
- no-connect marks 36 -> 38
Other:
- note added: "20 x 10k R\n2 x 1k R\n3 x 150 R\n1 x 220 R\n12 x QRE1113\n2 X NPN\n1 X PMOS\n1 X NMOS\n1 X MUX4051\n1 X MUX4052\n1 X RN-42\n1 X Tipka\n1 X Stikalo\n1 X LED\n2 X Motor, enkoder\n2 X MUX4051\n1 X Arduino Micro\n1 X Baterija 9V\n\n"
- note removed: "20 x 10k R\n2 x 1k R\n3 x 150 R\n2 x 300 R\n1 x 220 R\n12 x QRE1113\n4 X NPN\n1 X PMOS\n1 X NMOS\n1 X MUX4051\n1 X MUX4052\n1 X RN-42\n1 X Tipka\n1 X Stikalo\n3 X LED\n2 X Motor, enkoder\n2 X MUX4051\n1 X Arduino Micro\n1 X Baterija 9V\n\n"
- note removed: "LED"

Commit message: Narejen PCB
Parts:
- removed MUX4052_1: CD4052, symbol CD4052
- removed Q2: NPN, symbol Q_NPN_BCE
- removed R12: 1k, symbol R
- removed R13: 150, symbol R
- removed R14, R15, R16, R17: 10k, symbol R
- removed foto_senzor10, foto_senzor11, foto_senzor12, foto_senzor9: QRE1113, symbol QRE1113
- added J1, J2: ST_1x08, robot:ST_1x8, symbol Screw_Terminal_1x08
- ArduinoMicro1: footprint (none) -> robot:ArduinoMicro
- BT1: footprint (none) -> robot:Battery; symbol BATTERY -> BATTERY-RESCUE-robot
- BT2.1: footprint (none) -> RF_Modules:RN42
- C1, C2: footprint (none) -> Capacitors_ThroughHole:C_Rect_L4_W2.5_P2.5
- D1: footprint (none) -> Diodes_SMD:D_0603
- Driver1: footprint (none) -> Housings_DIP:DIP-16_W7.62mm_LongPads
- MUX4051_1: footprint (none) -> robot:CD4051
- MotorD1, MotorL1: footprint (none) -> robot:Motor
- Q1: footprint (none) -> TO_SOT_Packages_THT:TO-92_Inline_Narrow_Oval
- Q2: renamed from Q3; footprint (none) -> TO_SOT_Packages_THT:TO-220_Neutral123_Vertical
- Q3: renamed from Q4; footprint (none) -> robot:SOT-23
- R1, R10, R11, R2, R3, R4, R5, R6, R7, R8, R9: footprint (none) -> Resistors_SMD:R_0805_HandSoldering
- R12: renamed from R18; footprint (none) -> Resistors_SMD:R_0805_HandSoldering
- R13: renamed from R19; footprint (none) -> Resistors_SMD:R_0805_HandSoldering
- R14: renamed from R20; footprint (none) -> Resistors_SMD:R_0805_HandSoldering
- R15: renamed from R22; footprint (none) -> Resistors_SMD:R_0805_HandSoldering
- R16: renamed from R21; footprint (none) -> Resistors_SMD:R_0805_HandSoldering
- R17: renamed from R23; footprint (none) -> Resistors_SMD:R_0805_HandSoldering
- R18: renamed from R24; footprint (none) -> Resistors_SMD:R_0805_HandSoldering
- R19: renamed from R10k1; footprint (none) -> Resistors_SMD:R_0805_HandSoldering
- SW1: footprint (none) -> robot:Switch
- SW2: footprint (none) -> Buttons_Switches_ThroughHole:SW_PUSH_SMALL
- foto_senzor1, foto_senzor2, foto_senzor3, foto_senzor4, foto_senzor5, foto_senzor6, foto_senzor7, foto_senzor8: footprint (none) -> robot:QRE1113
Connections:
- net +5V: now also J1.7, J2.7
- net +9V: now also BT1.1, J1.8, J2.8; no longer BT1.~
- net A1: now also J1.6, J2.6
- net B1: now also J1.5, J2.5
- net C1: now also J1.4, J2.4
- net GND: now also BT1.2, J1.1, J2.1; no longer BT1.~
- net MUX1: now also J1.3, J2.3
- net ON/OFF: now also J1.2, J2.2
- net A2: no longer names the net of ArduinoMicro1.17 (D12)
- net B2: no longer names the net of ArduinoMicro1.18 (D13)
- net MUX2: no longer names the net of ArduinoMicro1.22 (A1)
- no-connect marks 38 -> 35
Other:
- note added: "18 x 10k R\n1 x 1k R\n3 x 150 R\n1 x 220 R\n12 x QRE1113\n1 X NPN\n1 X PMOS\n1 X NMOS\n1 X MUX4051\n1 X RN-42\n1 X Tipka\n1 X Stikalo\n1 X LED\n2 X Motor, enkoder\n2 X MUX4051\n1 X Arduino Micro\n1 X Baterija 9V\n\n"
- note removed: "20 x 10k R\n2 x 1k R\n3 x 150 R\n1 x 220 R\n12 x QRE1113\n2 X NPN\n1 X PMOS\n1 X NMOS\n1 X MUX4051\n1 X MUX4052\n1 X RN-42\n1 X Tipka\n1 X Stikalo\n1 X LED\n2 X Motor, enkoder\n2 X MUX4051\n1 X Arduino Micro\n1 X Baterija 9V\n\n"
- moved on the sheet: BT2.1, D1, Q2, Q3, R12, R13, R14, R15, R16, R17, R18, R19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
